Commit message: Changed some parameters

File: ros2_micromouse/urdf/micromouse.urdf (robot description, URDF)
Before this commit: robot micromouse, 5 links, 4 joints
Links:
- link base_link: mass 0.6 -> 0.1
- link left_wheel: mass 0.2 -> 0.1
- link right_wheel: mass 0.2 -> 0.1

Commit message: Added a LIDAR sensor

File: ros2_micromouse/urdf/micromouse.urdf (robot description, URDF)
Before this commit: robot micromouse, 5 links, 4 joints
Links:
- added link scan_link, mass 1e-4; collision box size=.01 .01 .01; visual box size=.01 .01 .01
Joints:
- added joint scan_joint: type fixed, parent base_link, child scan_link, origin xyz=0.0 0 0.02 rpy=0 0 0, axis 0 1 0

Commit message: Increased the size of the robot and the maze, provided a fix for the mapping

File: ros2_micromouse/urdf/micromouse.urdf (robot description, URDF)
Before this commit: robot micromouse, 6 links, 5 joints
Links:
- link base_link: mass 0.1 -> 12.5; geometry collision box size=0.435 0.225 0.15; collision sphere radius=0.0249
- link left_wheel: mass 0.1 -> 12.5; geometry collision cylinder length=.1 radius=.1; visual mesh filename=package://ros2_micromouse/meshes/robo_wheel.dae
- link right_wheel: mass 0.1 -> 12.5; geometry collision cylinder length=.1 radius=.1; visual mesh filename=package://ros2_micromouse/meshes/robo_wheel_right.dae
- link scan_link: geometry collision box size=.05 .05 .05; visual box size=.05 .05 .05
Joints:
- joint left_wheel_joint: origin xyz=0 0.0325 0 rpy=0 0 0 -> xyz=0 0.1625 0 rpy=0 0 0
- joint right_wheel_joint: origin xyz=0 -0.0325 0 rpy=0 0 0 -> xyz=0 -0.1625 0 rpy=0 0 0
- joint scan_joint: origin xyz=0.0 0 0.02 rpy=0 0 0 -> xyz=0.0 0 0.1 rpy=0 0 0
